Commit message: Proper vel. limits

File: python/6axis/robot.urdf (robot description, URDF)
Before this commit: robot onshape, 8 links, 7 joints
Joints:
- joint r1: limit lower=-2.96706 upper=2.96706 effort=1 velocity=20 -> lower=-2.96706 upper=2.96706 effort=1 velocity=1.75
- joint r2: limit lower=-2.44346 upper=1.13446 effort=1 velocity=20 -> lower=-2.44346 upper=1.13446 effort=1 velocity=1.57
- joint r3: limit lower=-3.14159 upper=1.22173 effort=1 velocity=20 -> lower=-3.14159 upper=1.22173 effort=1 velocity=1.57
- joint r4: limit lower=-5.23599 upper=5.23599 effort=1 velocity=20 -> lower=-5.23599 upper=5.23599 effort=1 velocity=2.62
- joint r5: limit lower=-2.26893 upper=2.26893 effort=1 velocity=20 -> lower=-2.26893 upper=2.26893 effort=1 velocity=2.1
- joint r6: limit lower=-5.23599 upper=5.23599 effort=1 velocity=20 -> lower=-5.23599 upper=5.23599 effort=1 velocity=3.32
