Commit message: Kinematics wip

File: python/sigmaban/robot.urdf (robot description, URDF)
Before this commit: robot onshape, 27 links, 26 joints
Joints:
- joint left_knee: limit effort=10 velocity=6 -> lower=0.0 upper=3.14 effort=10 velocity=6
- joint right_knee: limit effort=10 velocity=6 -> lower=0.0 upper=3.14 effort=10 velocity=6

Commit message: Removing test/comments in kinematics.py

File: python/sigmaban/robot.urdf (robot description, URDF)
Before this commit: robot onshape, 27 links, 26 joints
Joints:
- joint left_knee: limit lower=0.0 upper=3.14 effort=10 velocity=6 -> lower=0.05 upper=3.14 effort=10 velocity=6
- joint right_knee: limit lower=0.0 upper=3.14 effort=10 velocity=6 -> lower=0.05 upper=3.14 effort=10 velocity=6

Commit message: Updating Sigmaban model with joint limits

File: python/sigmaban/robot.urdf (robot description, URDF)
Before this commit: robot onshape, 27 links, 26 joints
Links:
- removed link left_foot_tip
- removed link right_foot_tip
- removed link vive_head
- added link left_foot, mass 1e-9
- added link right_foot, mass 1e-9
- link head__field_of_view_false: mass 0.137167 -> 0.120438
- link radius_v2: mass 0.133609 -> 0.120619
- link radius_v2_2: mass 0.133609 -> 0.120619
Joints:
- removed joint left_foot_tip_frame
- removed joint right_foot_tip_frame
- removed joint vive_head_frame
- added joint left_foot_frame: type fixed, parent left_foot_asm, child left_foot, origin xyz=0.06 6.45317e-16 -0.02033 rpy=8.38389e-16 -1.5708 0, axis 0 0 0
- added joint right_foot_frame: type fixed, parent right_foot_asm, child right_foot, origin xyz=0.06 1.02696e-15 -0.02033 rpy=4.64969e-19 -1.5708 0, axis 0 0 0
- joint camera_frame: origin xyz=-0.024933 0.0335 -0.0235 rpy=1.5708 -2.95668e-16 -1.5708 -> xyz=-0.024933 0.0335 -0.0235 rpy=3.14159 1.5708 0
- joint head_pitch: limit effort=10 velocity=6 -> lower=-0.785398 upper=1.5708 effort=10 velocity=6; origin xyz=-0.0235 1.04083e-16 0.058302 rpy=1.5708 -9.33402e-15 -1.5708 -> xyz=-0.0235 1.67921e-15 0.058302 rpy=1.5708 -5.26755e-18 -1.5708
- joint head_yaw: limit effort=10 velocity=6 -> lower=-2.0944 upper=2.0944 effort=10 velocity=6; origin xyz=0.035869 2.87964e-15 0.1595 rpy=1.00593e-14 2.25419e-14 -1.5708 -> xyz=0.035869 4.36359e-15 0.1595 rpy=3.46945e-16 2.84444e-15 -1.5708
- joint left_ankle_pitch: limit effort=10 velocity=6 -> lower=-1.5708 upper=1.5708 effort=10 velocity=6; origin xyz=-0.14 9.42128e-15 4.65253e-15 rpy=7.77156e-16 -8.97018e-15 -5.39997e-14 -> xyz=-0.14 9.46118e-15 4.71151e-15 rpy=-2.63106e-14 -1.45196e-14 -1.5669e-13
- joint left_ankle_roll: limit effort=10 velocity=6 -> lower=-0.785398 upper=0.785398 effort=10 velocity=6; origin xyz=-2.77556e-16 0.0201 0.016 rpy=1.5708 2.85175e-15 -3.14159 -> xyz=-2.22045e-16 0.0201 0.016 rpy=1.5708 7.53536e-19 3.14159
- joint left_elbow: limit effort=10 velocity=6 -> lower=-2.79253 upper=0 effort=10 velocity=6; origin xyz=0.0235 -0.142 -0.0025 rpy=-1.17212e-15 1.5708 0 -> xyz=0.0235 -0.142 -0.0025 rpy=1.63031e-15 1.5708 0
- joint left_hip_pitch: limit effort=10 velocity=6 -> lower=-1.5708 upper=1.5708 effort=10 velocity=6; origin xyz=-1.66533e-16 0.016 -0.0201 rpy=1.5708 -1.5708 0 -> xyz=1.38778e-16 0.016 -0.0201 rpy=1.5708 -1.56511 -9.4895e-13
- joint left_hip_roll: limit effort=10 velocity=6 -> lower=-0.523599 upper=0.523599 effort=10 velocity=6; origin xyz=2.35922e-16 -0.0200991 -0.0604 rpy=1.5708 -1.5708 0 -> xyz=-1.11022e-16 -0.0200991 -0.0604 rpy=1.5708 -1.5708 0
- joint left_hip_yaw: limit effort=10 velocity=6 -> lower=-1.0472 upper=1.0472 effort=10 velocity=6; origin xyz=0.00586897 0.0464 -0.0411 rpy=-1.82465e-15 -3.03444e-15 1.5708 -> xyz=0.00586897 0.0464 -0.0411 rpy=1.43162e-16 -2.2295e-14 1.5708
- joint left_knee: limit lower=0.05 upper=3.14 effort=10 velocity=6 -> lower=0. upper=3.14159 effort=10 velocity=6; origin xyz=-5.21284e-16 0.14 -0.001 rpy=5.28137e-15 7.03032e-15 -1.5708 -> xyz=-7.5287e-16 0.14 -0.001 rpy=1.92498e-15 1.2611e-14 -1.5708
- joint left_shoulder_pitch: limit effort=10 velocity=6 -> lower=-2.18166 upper=2.18166 effort=10 velocity=6; origin xyz=0.030869 0.0795 0.143 rpy=-1.5708 1.58669e-15 1.2761e-15 -> xyz=0.030869 0.0795 0.143 rpy=-1.5708 -7.21645e-15 2.48831e-15
- joint left_shoulder_roll: limit effort=10 velocity=6 -> lower=-0.0872665 upper=1.5708 effort=10 velocity=6
- joint right_ankle_pitch: limit effort=10 velocity=6 -> lower=-1.5708 upper=1.5708 effort=10 velocity=6; origin xyz=-0.14 -1.52768e-14 5.05741e-14 rpy=-4.44089e-16 -2.94225e-15 3.03503e-14 -> xyz=-0.14 -1.56732e-14 5.03798e-14 rpy=-4.4409e-16 -4.49305e-15 1.11963e-13
- joint right_ankle_roll: limit effort=10 velocity=6 -> lower=-0.785398 upper=0.785398 effort=10 velocity=6; origin xyz=-3.33067e-16 0.0201 -0.016 rpy=1.5708 -3.91365e-15 3.14159 -> xyz=-2.22045e-16 0.0201 -0.016 rpy=1.5708 4.64969e-19 -3.14159
- joint right_elbow: limit effort=10 velocity=6 -> lower=-2.79253 upper=-0 effort=10 velocity=6
- joint right_hip_pitch: limit effort=10 velocity=6 -> lower=-1.5708 upper=1.5708 effort=10 velocity=6; origin xyz=0.000235943 -0.016 -0.0201 rpy=1.5708 -1.5708 0 -> xyz=0.000235943 -0.016 -0.0201 rpy=1.5708 -1.56511 -2.92366e-13
- joint right_hip_roll: limit effort=10 velocity=6 -> lower=-0.523599 upper=0.523599 effort=10 velocity=6; origin xyz=-2.498e-16 -0.0200991 -0.0604 rpy=1.5708 -1.5708 0 -> xyz=6.245e-17 -0.0200991 -0.0604 rpy=1.5708 -1.5708 0
- joint right_hip_yaw: limit effort=10 velocity=6 -> lower=-1.0472 upper=1.0472 effort=10 velocity=6; origin xyz=0.00586897 -0.0464 -0.0411 rpy=2.16251e-14 -1.98167e-15 1.5708 -> xyz=0.00586897 -0.0464 -0.0411 rpy=1.22835e-15 -2.11957e-15 1.5708
- joint right_knee: limit lower=0.05 upper=3.14 effort=10 velocity=6 -> lower=0. upper=3.14159 effort=10 velocity=6; origin xyz=-1.17094e-16 0.14 -2.05669e-14 rpy=1.27676e-15 -1.58087e-15 -1.5708 -> xyz=-3.81639e-17 0.14 -2.05357e-14 rpy=-1.24994e-15 -5.32933e-16 -1.5708
- joint right_shoulder_pitch: limit effort=10 velocity=6 -> lower=-2.18166 upper=2.18166 effort=10 velocity=6; origin xyz=0.030869 -0.0795 0.143 rpy=1.5708 -4.80171e-15 3.14159 -> xyz=0.030869 -0.0795 0.143 rpy=1.5708 -1.84019e-14 3.14159
- joint right_shoulder_roll: limit effort=10 velocity=6 -> lower=-1.5708 upper=0.0872665 effort=10 velocity=6; origin xyz=-0.0235 -0.03 -0.035 rpy=-3.60822e-16 -1.5708 0 -> xyz=-0.0235 -0.03 -0.035 rpy=-3.58863e-16 -1.5708 0
- joint trunk_frame: origin xyz=0.00586803 -3.83374e-15 -0.1015 rpy=2.59035e-15 -1.04919e-28 -6.69483e-15 -> xyz=0.00586803 -3.58583e-15 -0.1015 rpy=-2.22624e-15 4.13778e-27 -1.14065e-13

Commit message: Wip

File: python/sigmaban/robot.urdf (robot description, URDF)
Before this commit: robot onshape, 26 links, 25 joints
Links:
- link head__field_of_view_false: mass 0.120438 -> 0.249938
- link left_humerus: mass 0.111948 -> 0.241448
- link mx106_with_u_l: mass 0.136461 -> 0.421574
- link mx106_with_u_l_2: mass 0.136461 -> 0.421574
- link mx106_with_u_r: mass 0.136461 -> 0.421574
- link mx106_with_u_r_2: mass 0.136461 -> 0.421574
- link radius_v2: mass 0.120619 -> 0.250119
- link radius_v2_2: mass 0.120619 -> 0.250119
- link right_humerus: mass 0.111948 -> 0.241448
- link thigh_horn_left: mass 0.0845547 -> 0.227111
- link thigh_horn_right: mass 0.0845547 -> 0.227111
- link torso: mass 1.74256 -> 2.39006
Joints:
- joint head_pitch: origin xyz=-0.0235 1.67921e-15 0.058302 rpy=1.5708 -5.26755e-18 -1.5708 -> xyz=-0.0235 1.63064e-15 0.058302 rpy=1.5708 -5.26755e-18 -1.5708
- joint head_yaw: origin xyz=0.035869 4.36359e-15 0.1595 rpy=3.46945e-16 2.84444e-15 -1.5708 -> xyz=0.035869 2.46254e-15 0.1595 rpy=4.02456e-16 -2.25859e-14 -1.5708
- joint left_ankle_pitch: origin xyz=-0.14 9.46118e-15 4.71151e-15 rpy=-2.63106e-14 -1.45196e-14 -1.5669e-13 -> xyz=-0.14 8.93643e-15 -4.26742e-15 rpy=6.00611e-15 -4.79034e-15 -6.38113e-14
- joint left_ankle_roll: origin xyz=-2.22045e-16 0.0201 0.016 rpy=1.5708 7.53536e-19 3.14159 -> xyz=-2.22045e-16 0.0201 0.016 rpy=1.5708 -4.79033e-15 -3.14159
- joint left_foot_frame: origin xyz=0.06 6.45317e-16 -0.02033 rpy=8.38389e-16 -1.5708 0 -> xyz=0.06 0.0055 -0.00483 rpy=3.04574e-27 -1.5708 0
- joint left_hip_pitch: origin xyz=1.38778e-16 0.016 -0.0201 rpy=1.5708 -1.56511 -9.4895e-13 -> xyz=-2.08167e-16 0.016 -0.0201 rpy=1.5708 -1.56511 8.40664e-12
- joint left_hip_roll: origin xyz=-1.11022e-16 -0.0200991 -0.0604 rpy=1.5708 -1.5708 0 -> xyz=-1.17961e-16 -0.0200991 -0.0604 rpy=1.5708 -1.5708 0
- joint left_hip_yaw: origin xyz=0.00586897 0.0464 -0.0411 rpy=1.43162e-16 -2.2295e-14 1.5708 -> xyz=0.00586897 0.0464 -0.0411 rpy=1.38778e-17 -2.2295e-14 1.5708
- joint left_knee: limit lower=0. upper=3.14159 effort=10 velocity=6 -> lower=0 upper=3.14159 effort=10 velocity=6; origin xyz=-7.5287e-16 0.14 -0.001 rpy=1.92498e-15 1.2611e-14 -1.5708 -> xyz=4.11129e-16 0.14 -0.001 rpy=-1.18197e-15 -3.78471e-15 -1.5708
- joint right_ankle_pitch: origin xyz=-0.14 -1.56732e-14 5.03798e-14 rpy=-4.4409e-16 -4.49305e-15 1.11963e-13 -> xyz=-0.14 -1.56316e-14 -2.08167e-17 rpy=1.46503e-15 -5.21573e-15 -5.73004e-19
- joint right_ankle_roll: origin xyz=-2.22045e-16 0.0201 -0.016 rpy=1.5708 4.64969e-19 -3.14159 -> xyz=2.77556e-16 0.0201 -0.016 rpy=1.5708 -1.43631e-15 3.14159
- joint right_foot_frame: origin xyz=0.06 1.02696e-15 -0.02033 rpy=4.64969e-19 -1.5708 0 -> xyz=0.06 -0.0055 -0.00483 rpy=-1.661e-16 -1.5708 0
- joint right_hip_pitch: origin xyz=0.000235943 -0.016 -0.0201 rpy=1.5708 -1.56511 -2.92366e-13 -> xyz=0.000235943 -0.016 -0.0201 rpy=1.5708 -1.56511 -2.04106e-13
- joint right_hip_roll: origin xyz=6.245e-17 -0.0200991 -0.0604 rpy=1.5708 -1.5708 0 -> xyz=4.85723e-17 -0.0200991 -0.0604 rpy=1.5708 -1.5708 0
- joint right_hip_yaw: origin xyz=0.00586897 -0.0464 -0.0411 rpy=1.22835e-15 -2.11957e-15 1.5708 -> xyz=0.00586897 -0.0464 -0.0411 rpy=1.08941e-15 -2.22601e-15 1.5708
- joint right_knee: limit lower=0. upper=3.14159 effort=10 velocity=6 -> lower=-0 upper=3.14159 effort=10 velocity=6; origin xyz=-3.81639e-17 0.14 -2.05357e-14 rpy=-1.24994e-15 -5.32933e-16 -1.5708 -> xyz=3.05311e-16 0.14 -2.01748e-14 rpy=-5.68163e-14 -6.87273e-16 -1.5708
- joint right_shoulder_roll: origin xyz=-0.0235 -0.03 -0.035 rpy=-3.58863e-16 -1.5708 0 -> xyz=-0.0235 -0.03 -0.035 rpy=-5.55112e-17 -1.5708 0
- joint trunk_frame: origin xyz=0.00586803 -3.58583e-15 -0.1015 rpy=-2.22624e-15 4.13778e-27 -1.14065e-13 -> xyz=0.00586803 -3.95579e-15 -0.1015 rpy=2.09431e-15 2.18595e-26 -4.72596e-14
