Commit message: Fixing the model, adding gravity compensation calculation

File: python/sigmaban/robot.urdf (robot description, URDF)
Before this commit: robot onshape, 26 links, 25 joints
Links:
- link head__field_of_view_false: mass 0.249938 -> 0.22740577538449363582; geometry collision box size=0.040199999999999999623 0.061100000000000001532 0.041000000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; collision box size=0.061600000000000001976 0.047000000000000000111 0.003000000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
- link left_foot_asm: mass 0.32139 -> 0.32138977066764801149; geometry collision box size=0.091999999999999998446 0.1575999999999999901 0.00300000000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; collision cylinder length=0.016000000000000000333 radius=0.0080000000000000001665
- link left_humerus: mass 0.241448 -> 0.21891648912829692053; geometry collision box size=0.040199999999999999623 0.061100000000000001532 0.041000000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; visual box size=0.040199999999999999623 0.061100000000000001532 0.041000000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
- link mx106_with_u_l: mass 0.421574 -> 0.42157376486091741041; geometry collision box size=0.026999999999999999695 0.058000000000000002942 0.025999999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; collision box size=0.026999999999999999695 0.058000000000000002942 0.025999999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
- link mx106_with_u_l_2: mass 0.421574 -> 0.4215737648609173549; geometry collision box size=0.026999999999999999695 0.058000000000000002942 0.025999999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; collision box size=0.026999999999999999695 0.058000000000000002942 0.025999999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
- link mx106_with_u_r: mass 0.421574 -> 0.4215737648609173549; geometry collision box size=0.026999999999999999695 0.058000000000000002942 0.025999999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; collision box size=0.026999999999999999695 0.058000000000000002942 0.025999999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
- link mx106_with_u_r_2: mass 0.421574 -> 0.4215737648609173549; geometry collision box size=0.026999999999999999695 0.058000000000000002942 0.025999999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; collision box size=0.026999999999999999695 0.058000000000000002942 0.025999999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
- link radius_v2: mass 0.250119 -> 0.22758681850404099967; geometry collision box size=0.040199999999999999623 0.061100000000000001532 0.041000000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; collision box size=0.077551200000000000689 0.041200000000000000511 0.003000000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
- link radius_v2_2: mass 0.250119 -> 0.22758681850404099967; geometry collision box size=0.040199999999999999623 0.061100000000000001532 0.041000000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; collision box size=0.077551200000000000689 0.041200000000000000511 0.003000000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
- link right_foot_asm: mass 0.32139 -> 0.32138977066764795598; geometry collision box size=0.091999999999999998446 0.1575999999999999901 0.00300000000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; collision cylinder length=0.016000000000000000333 radius=0.0080000000000000001665
- link right_humerus: mass 0.241448 -> 0.21891648912829692053; geometry collision box size=0.040199999999999999623 0.061100000000000001532 0.041000000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; visual box size=0.040199999999999999623 0.061100000000000001532 0.041000000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
- link thigh_horn_left: mass 0.227111 -> 0.22711106780187376164; geometry collision box size=0.026999999999999999695 0.058000000000000002942 0.025999999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; collision box size=0.02999999999999999889 0.080000000000000001665 0.0030000000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
- link thigh_horn_right: mass 0.227111 -> 0.22711106780187373388; geometry collision box size=0.026999999999999999695 0.058000000000000002942 0.025999999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; collision box size=0.02999999999999999889 0.080000000000000001665 0.0030000000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
- link tibia_left_full: mass 0.0501468 -> 0.050146782973123575633; geometry collision box size=0.14999999999999999445 0.035000000000000003331 0.0030000000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; collision box size=0.14999999999999999445 0.035000000000000003331 0.0030000000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
- link tibia_right_full: mass 0.0501468 -> 0.050146782973123575633; geometry collision box size=0.14999999999999999445 0.035000000000000003331 0.0030000000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; collision box size=0.14999999999999999445 0.035000000000000003331 0.0030000000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
- link torso: mass 2.39006 -> 2.3224634991401664763; geometry collision box size=0.040199999999999999623 0.061100000000000001532 0.041000000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; collision box size=0.040199999999999999623 0.061100000000000001532 0.041000000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
- link u_hip_with_saver: mass 0.136031 -> 0.13603079497559261712
- link u_hip_with_saver_2: mass 0.136031 -> 0.13603079497559264488
- link u_neck: mass 0.0544799 -> 0.054479900613359215356; geometry collision box size=0.02999999999999999889 0.065802000000000013258 0.0030000000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; collision box size=0.02999999999999999889 0.065802000000000013258 0.0030000000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
- link u_shoulder: mass 0.0570101 -> 0.057010148283040865125; geometry collision box size=0.049000000000000001887 0.02999999999999999889 0.0062500000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; visual box size=0.049000000000000001887 0.02999999999999999889 0.0062500000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
- link u_shoulder_2: mass 0.0570101 -> 0.057010148283040872064; geometry collision box size=0.049000000000000001887 0.02999999999999999889 0.0062500000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; visual box size=0.049000000000000001887 0.02999999999999999889 0.0062500000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
Joints:
- joint camera_frame: origin xyz=-0.024933 0.0335 -0.0235 rpy=3.14159 1.5708 0 -> xyz=-0.024933000004023209151 0.033500000000054735994 -0.023500000000009093476 rpy=3.1415926535897797933 1.5707963267948958919 0
- joint head_base_frame: origin xyz=0.035869 2.87859e-15 0.1595 rpy=3.79641e-14 -9.95037e-15 -1.04223e-13 -> xyz=0.035868973494361730547 2.8785898342325425989e-15 0.15950000000001055001 rpy=3.7964142151183067762e-14 -9.9503738582029639158e-15 -1.0422282733566275005e-13
- joint head_pitch: limit lower=-0.785398 upper=1.5708 effort=10 velocity=6 -> lower=-0.785398163397448279 upper=1.570796326794896558 effort=10 velocity=6; origin xyz=-0.0235 1.63064e-15 0.058302 rpy=1.5708 -5.26755e-18 -1.5708 -> xyz=-0.023499999999997519401 2.2482016248659419944e-15 0.058302041851018837626 rpy=1.5707963267948794606 -9.3778577129540909355e-15 -1.5707963267950493247
- joint head_yaw: limit lower=-2.0944 upper=2.0944 effort=10 velocity=6 -> lower=-2.0943951023931952626 upper=2.0943951023931952626 effort=10 velocity=6; origin xyz=0.035869 2.46254e-15 0.1595 rpy=4.02456e-16 -2.25859e-14 -1.5708 -> xyz=0.035868973494361702792 -2.0768736888402729908e-15 0.15950000000001013367 rpy=9.7750460134011636162e-15 -1.1951368418674699747e-14 -1.5707963267948004127
- joint left_ankle_pitch: limit lower=-1.5708 upper=1.5708 effort=10 velocity=6 -> lower=-1.570796326794896558 upper=1.570796326794896558 effort=10 velocity=6; origin xyz=-0.14 8.93643e-15 -4.26742e-15 rpy=6.00611e-15 -4.79034e-15 -6.38113e-14 -> xyz=-0.14000000000002504885 1.3950646193805482653e-14 0 rpy=-6.1231560962847779576e-14 -1.8582018332858367343e-14 -5.6936840381678493267e-14
- joint left_ankle_roll: limit lower=-0.785398 upper=0.785398 effort=10 velocity=6 -> lower=-0.785398163397448279 upper=0.785398163397448279 effort=10 velocity=6; origin xyz=-2.22045e-16 0.0201 0.016 rpy=1.5708 -4.79033e-15 -3.14159 -> xyz=-1.1102230246251565404e-16 0.020099999999999937361 0.016000000000000135641 rpy=1.5707963267948934494 6.5049045633606117685e-15 3.1415926535897895633
- joint left_elbow: limit lower=-2.79253 upper=0 effort=10 velocity=6 -> lower=-2.7925268031909271649 upper=0 effort=10 velocity=6; origin xyz=0.0235 -0.142 -0.0025 rpy=1.63031e-15 1.5708 0 -> xyz=0.02349999999999953515 -0.14200000000002568901 -0.0024999999999900518466 rpy=1.6303130422869307442e-15 1.570796326794896336 0
- joint left_foot_frame: origin xyz=0.06 0.0055 -0.00483 rpy=3.04574e-27 -1.5708 0 -> xyz=0.060000000000000275335 0.0055000000000001159073 -0.0048299999999999489175 rpy=-6.2664175067465104603e-16 -1.5707963267948947816 0
- joint left_hip_pitch: limit lower=-1.5708 upper=1.5708 effort=10 velocity=6 -> lower=-1.570796326794896558 upper=1.570796326794896558 effort=10 velocity=6; origin xyz=-2.08167e-16 0.016 -0.0201 rpy=1.5708 -1.56511 8.40664e-12 -> xyz=-1.8041124150158793782e-16 0.016000000000000000333 -0.020099999999999784706 rpy=1.57079632679489678 -1.5707963267948910069 0
- joint left_hip_roll: limit lower=-0.523599 upper=0.523599 effort=10 velocity=6 -> lower=-0.52359877559829881566 upper=0.52359877559829881566 effort=10 velocity=6; origin xyz=-1.17961e-16 -0.0200991 -0.0604 rpy=1.5708 -1.5708 0 -> xyz=-8.3266726846886740532e-17 -0.020099054048956847135 -0.060400000000000342304 rpy=1.5707963267948823471 -1.5707963267948934494 0
- joint left_hip_yaw: limit lower=-1.0472 upper=1.0472 effort=10 velocity=6 -> lower=-1.0471975511965976313 upper=1.0471975511965976313 effort=10 velocity=6; origin xyz=0.00586897 0.0464 -0.0411 rpy=1.38778e-17 -2.2295e-14 1.5708 -> xyz=0.0058689734943615417054 0.04640000000001042596 -0.041099999999999782541 rpy=2.3786004854476977408e-16 -4.9676806335296454892e-15 1.5707963267948459318
- joint left_knee: limit lower=0 upper=3.14159 effort=10 velocity=6 -> lower=0 upper=3.141592653589793116 effort=10 velocity=6; origin xyz=4.11129e-16 0.14 -0.001 rpy=-1.18197e-15 -3.78471e-15 -1.5708 -> xyz=-2.3678975447083416839e-16 0.13999999999999973577 2.0757701113538473692e-14 rpy=2.8102530281515361041e-15 3.8106870795519192501e-15 -1.5707963267948208408
- joint left_shoulder_pitch: limit lower=-2.18166 upper=2.18166 effort=10 velocity=6 -> lower=-2.1816615649929120835 upper=2.1816615649929120835 effort=10 velocity=6; origin xyz=0.030869 0.0795 0.143 rpy=-1.5708 -7.21645e-15 2.48831e-15 -> xyz=0.03086897349438466609 0.079500000000020845659 0.14300000000001039657 rpy=-1.5707963267949047736 -7.2164496600635995543e-15 2.4883110829860584224e-15
- joint left_shoulder_roll: limit lower=-0.0872665 upper=1.5708 effort=10 velocity=6 -> lower=-0.087266462599716473902 upper=1.570796326794896558 effort=10 velocity=6; origin xyz=0.0235 0.03 0.035 rpy=-3.14159 -1.5708 0 -> xyz=0.023500000000000003525 0.030000000000000054401 0.034999999999999933942 rpy=-3.1415926535897917837 -1.5707963267948958919 0
- joint right_ankle_pitch: limit lower=-1.5708 upper=1.5708 effort=10 velocity=6 -> lower=-1.570796326794896558 upper=1.570796326794896558 effort=10 velocity=6; origin xyz=-0.14 -1.56316e-14 -2.08167e-17 rpy=1.46503e-15 -5.21573e-15 -5.73004e-19 -> xyz=-0.14000000000024515057 -1.5889199678209564581e-14 3.0114799542957371159e-14 rpy=5.0446957243049974607e-16 -6.5007295419637772327e-15 -1.5612511284079219651e-17
- joint right_ankle_roll: limit lower=-0.785398 upper=0.785398 effort=10 velocity=6 -> lower=-0.785398163397448279 upper=0.785398163397448279 effort=10 velocity=6; origin xyz=2.77556e-16 0.0201 -0.016 rpy=1.5708 -1.43631e-15 3.14159 -> xyz=3.8857805861880478915e-16 0.020099999999999926953 -0.015999999999999691552 rpy=1.570796326794896336 2.4094412794995258621e-15 3.1415926535897926719
- joint right_elbow: limit lower=-2.79253 upper=-0 effort=10 velocity=6 -> lower=-2.7925268031909271649 upper=-0 effort=10 velocity=6; origin xyz=-0.0235 -0.142 -0.0025 rpy=3.14159 -1.5708 0 -> xyz=-0.023500000000009860224 -0.14200000000001986034 -0.0024999999999998911981 rpy=3.141592653589793116 -1.5707963267948954478 0
- joint right_foot_frame: origin xyz=0.06 -0.0055 -0.00483 rpy=-1.661e-16 -1.5708 0 -> xyz=0.05999999999999905409 -0.005500000000000331013 -0.0048299999999974474463 rpy=5.2020940636638788206e-15 -1.570796326794891451 0
- joint right_hip_pitch: limit lower=-1.5708 upper=1.5708 effort=10 velocity=6 -> lower=-1.570796326794896558 upper=1.570796326794896558 effort=10 velocity=6; origin xyz=0.000235943 -0.016 -0.0201 rpy=1.5708 -1.56511 -2.04106e-13 -> xyz=0.00023594338595557540206 -0.01599999999999995523 -0.020100000000000020628 rpy=1.5707963267949038855 -1.5707963267948861219 0
- joint right_hip_roll: limit lower=-0.523599 upper=0.523599 effort=10 velocity=6 -> lower=-0.52359877559829881566 upper=0.52359877559829881566 effort=10 velocity=6; origin xyz=4.85723e-17 -0.0200991 -0.0604 rpy=1.5708 -1.5708 0 -> xyz=4.8572257327350598644e-17 -0.020099054048955403845 -0.06039999999999973862 rpy=1.5707963267949003328 -1.5707963267948901187 0
- joint right_hip_yaw: limit lower=-1.0472 upper=1.0472 effort=10 velocity=6 -> lower=-1.0471975511965976313 upper=1.0471975511965976313 effort=10 velocity=6; origin xyz=0.00586897 -0.0464 -0.0411 rpy=1.08941e-15 -2.22601e-15 1.5708 -> xyz=0.0058689734943568345332 -0.046400000000004472389 -0.041099999999999956013 rpy=3.9664277854914981584e-16 -5.2373734976912576551e-15 1.5707963267948397146
- joint right_knee: limit lower=-0 upper=3.14159 effort=10 velocity=6 -> lower=-0 upper=3.141592653589793116 effort=10 velocity=6; origin xyz=3.05311e-16 0.14 -2.01748e-14 rpy=-5.68163e-14 -6.87273e-16 -1.5708 -> xyz=-2.9143354396410359186e-16 0.14000000000000067946 -9.5756735873919751612e-16 rpy=-3.9621086151768392032e-15 7.7674449885245198315e-16 -1.5707963267948938935
- joint right_shoulder_pitch: limit lower=-2.18166 upper=2.18166 effort=10 velocity=6 -> lower=-2.1816615649929120835 upper=2.1816615649929120835 effort=10 velocity=6; origin xyz=0.030869 -0.0795 0.143 rpy=1.5708 -1.84019e-14 3.14159 -> xyz=0.03086897349437638105 -0.079500000000014198198 0.14300000000001014677 rpy=1.5707963267948708008 -1.8374191057546290257e-14 3.141592653589783346
- joint right_shoulder_roll: limit lower=-1.5708 upper=0.0872665 effort=10 velocity=6 -> lower=-1.570796326794896558 upper=0.087266462599716473902 effort=10 velocity=6; origin xyz=-0.0235 -0.03 -0.035 rpy=-5.55112e-17 -1.5708 0 -> xyz=-0.023500000000005155654 -0.029999999999999651945 -0.034999999999995798361 rpy=-8.8817841970007218144e-16 -1.5707963267948961139 0
- joint trunk_frame: origin xyz=0.00586803 -3.95579e-15 -0.1015 rpy=2.09431e-15 2.18595e-26 -4.72596e-14 -> xyz=0.0058680275433158485265 -3.9238251073735071353e-15 -0.10150000000000060363 rpy=5.5093833584565697626e-15 4.4079575231487197359e-25 -5.958092587816837932e-14
