Commit message: Reorganizing python/ directory a little bit (wip)

File: python/sigmaban/robot.urdf (robot description, URDF)
Before this commit: robot onshape, 26 links, 25 joints
Links:
- link head__field_of_view_false: geometry collision box size=0.040199999999999999623 0.061100000000000001532 0.041000000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; collision box size=0.061600000000000001976 0.047000000000000000111 0.003000000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
- link left_foot_asm: geometry collision box size=0.091999999999999998446 0.1575999999999999901 0.00300000000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; collision cylinder length=0.016000000000000000333 radius=0.0080000000000000001665
- link left_humerus: geometry collision box size=0.040199999999999999623 0.061100000000000001532 0.041000000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; visual mesh filename=package:///left_humerus_visual.stl
- link mx106_with_u_l: mass 0.42157376486091741041 -> 0.13646106366842530866; geometry collision box size=0.026999999999999999695 0.058000000000000002942 0.025999999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; collision box size=0.026999999999999999695 0.058000000000000002942 0.025999999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
- link mx106_with_u_l_2: mass 0.4215737648609173549 -> 0.13646106366842530866; geometry collision box size=0.026999999999999999695 0.058000000000000002942 0.025999999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; collision box size=0.026999999999999999695 0.058000000000000002942 0.025999999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
- link mx106_with_u_r: mass 0.4215737648609173549 -> 0.13646106366842530866; geometry collision box size=0.026999999999999999695 0.058000000000000002942 0.025999999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; collision box size=0.026999999999999999695 0.058000000000000002942 0.025999999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
- link mx106_with_u_r_2: mass 0.4215737648609173549 -> 0.13646106366842530866; geometry collision box size=0.026999999999999999695 0.058000000000000002942 0.025999999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; collision box size=0.026999999999999999695 0.058000000000000002942 0.025999999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
- link radius_v2: geometry collision box size=0.040199999999999999623 0.061100000000000001532 0.041000000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; collision box size=0.077551200000000000689 0.041200000000000000511 0.003000000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
- link radius_v2_2: geometry collision box size=0.040199999999999999623 0.061100000000000001532 0.041000000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; collision box size=0.077551200000000000689 0.041200000000000000511 0.003000000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
- link right_foot_asm: geometry collision box size=0.091999999999999998446 0.1575999999999999901 0.00300000000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; collision cylinder length=0.016000000000000000333 radius=0.0080000000000000001665
- link right_humerus: geometry collision box size=0.040199999999999999623 0.061100000000000001532 0.041000000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; visual mesh filename=package:///right_humerus_visual.stl
- link thigh_horn_left: mass 0.22711106780187376164 -> 0.084554717205627710763; geometry collision box size=0.026999999999999999695 0.058000000000000002942 0.025999999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; collision box size=0.02999999999999999889 0.080000000000000001665 0.0030000000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
- link thigh_horn_right: mass 0.22711106780187373388 -> 0.084554717205627710763; geometry collision box size=0.026999999999999999695 0.058000000000000002942 0.025999999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; collision box size=0.02999999999999999889 0.080000000000000001665 0.0030000000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
- link tibia_left_full: geometry collision box size=0.14999999999999999445 0.035000000000000003331 0.0030000000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; collision box size=0.14999999999999999445 0.035000000000000003331 0.0030000000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
- link tibia_right_full: geometry collision box size=0.14999999999999999445 0.035000000000000003331 0.0030000000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; collision box size=0.14999999999999999445 0.035000000000000003331 0.0030000000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
- link torso: geometry collision box size=0.040199999999999999623 0.061100000000000001532 0.041000000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; collision box size=0.040199999999999999623 0.061100000000000001532 0.041000000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
- link u_neck: geometry collision box size=0.02999999999999999889 0.065802000000000013258 0.0030000000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; collision box size=0.02999999999999999889 0.065802000000000013258 0.0030000000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
- link u_shoulder: geometry collision box size=0.049000000000000001887 0.02999999999999999889 0.0062500000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; visual mesh filename=package:///u_shoulder_visual.stl
- link u_shoulder_2: geometry collision box size=0.049000000000000001887 0.02999999999999999889 0.0062500000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; visual mesh filename=package:///u_shoulder_2_visual.stl
Joints:
- joint camera_frame: origin xyz=-0.024933000004023209151 0.033500000000054735994 -0.023500000000009093476 rpy=3.1415926535897797933 1.5707963267948958919 0 -> xyz=-0.02493300000402396549 0.033500000000056068261 -0.023500000000011109225 rpy=-3.1415926535897855665 1.5707963267948905628 0
- joint head_pitch: limit lower=-0.785398163397448279 upper=1.570796326794896558 effort=10 velocity=6 -> effort=10 velocity=6; origin xyz=-0.023499999999997519401 2.2482016248659419944e-15 0.058302041851018837626 rpy=1.5707963267948794606 -9.3778577129540909355e-15 -1.5707963267950493247 -> xyz=-0.023500000000001953354 1.0408340855860842566e-16 0.058302041851018782115 rpy=1.570796326794881459 -9.3340175461126013445e-15 -1.5707963267949771602
- joint head_yaw: limit lower=-2.0943951023931952626 upper=2.0943951023931952626 effort=10 velocity=6 -> effort=10 velocity=6; origin xyz=0.035868973494361702792 -2.0768736888402729908e-15 0.15950000000001013367 rpy=9.7750460134011636162e-15 -1.1951368418674699747e-14 -1.5707963267948004127 -> xyz=0.035868973494361661158 2.8796409701214989879e-15 0.15950000000001055001 rpy=1.0059319781662864725e-14 2.2541937107368225271e-14 -1.570796326795006026
- joint left_ankle_pitch: limit lower=-1.570796326794896558 upper=1.570796326794896558 effort=10 velocity=6 -> effort=10 velocity=6; origin xyz=-0.14000000000002504885 1.3950646193805482653e-14 0 rpy=-6.1231560962847779576e-14 -1.8582018332858367343e-14 -5.6936840381678493267e-14 -> xyz=-0.13999999999999410139 9.4230179215060161368e-15 4.6629367034256574698e-15 rpy=6.6613381477670753924e-16 -8.970180271625489804e-15 -5.3999664202879601807e-14
- joint left_ankle_roll: limit lower=-0.785398163397448279 upper=0.785398163397448279 effort=10 velocity=6 -> effort=10 velocity=6; origin xyz=-1.1102230246251565404e-16 0.020099999999999937361 0.016000000000000135641 rpy=1.5707963267948934494 6.5049045633606117685e-15 3.1415926535897895633 -> xyz=-3.3306690738754696213e-16 0.020100000000000041445 0.015999999999999917066 rpy=1.5707963267948990005 2.8517487916724881289e-15 -3.1415926535897926719
- joint left_elbow: limit lower=-2.7925268031909271649 upper=0 effort=10 velocity=6 -> effort=10 velocity=6; origin xyz=0.02349999999999953515 -0.14200000000002568901 -0.0024999999999900518466 rpy=1.6303130422869307442e-15 1.570796326794896336 0 -> xyz=0.023499999999999174327 -0.14200000000002915845 -0.0024999999999899061298 rpy=-1.1721201801673205241e-15 1.5707963267948961139 0
- joint left_foot_frame: origin xyz=0.060000000000000275335 0.0055000000000001159073 -0.0048299999999999489175 rpy=-6.2664175067465104603e-16 -1.5707963267948947816 0 -> xyz=0.059999999999999109601 5.3429483060085658508e-16 -0.02033000000000043106 rpy=-2.775557561558958448e-17 -1.570796326794891451 0
- joint left_hip_pitch: limit lower=-1.570796326794896558 upper=1.570796326794896558 effort=10 velocity=6 -> effort=10 velocity=6; origin xyz=-1.8041124150158793782e-16 0.016000000000000000333 -0.020099999999999784706 rpy=1.57079632679489678 -1.5707963267948910069 0 -> xyz=-1.8041124150158793782e-16 0.016000000000000007272 -0.020099999999999802053 rpy=1.5707963267948976682 -1.5707963267948936714 0
- joint left_hip_roll: limit lower=-0.52359877559829881566 upper=0.52359877559829881566 effort=10 velocity=6 -> effort=10 velocity=6; origin xyz=-8.3266726846886740532e-17 -0.020099054048956847135 -0.060400000000000342304 rpy=1.5707963267948823471 -1.5707963267948934494 0 -> xyz=2.3592239273284576484e-16 -0.020099054048956215696 -0.060399999999998552069 rpy=1.5707963267948876762 -1.5707963267948923392 0
- joint left_hip_yaw: limit lower=-1.0471975511965976313 upper=1.0471975511965976313 effort=10 velocity=6 -> effort=10 velocity=6; origin xyz=0.0058689734943615417054 0.04640000000001042596 -0.041099999999999782541 rpy=2.3786004854476977408e-16 -4.9676806335296454892e-15 1.5707963267948459318 -> xyz=0.0058689734943615451748 0.04640000000001042596 -0.04109999999999978948 rpy=-1.824649325745780325e-15 -3.0483134745539648229e-15 1.5707963267949009989
- joint left_knee: limit lower=0 upper=3.141592653589793116 effort=10 velocity=6 -> effort=10 velocity=6; origin xyz=-2.3678975447083416839e-16 0.13999999999999973577 2.0757701113538473692e-14 rpy=2.8102530281515361041e-15 3.8106870795519192501e-15 -1.5707963267948208408 -> xyz=-5.1521287236511170704e-16 0.13999999999999945821 -0.00099999999997956584563 rpy=5.6066262743583744929e-15 6.7205214539759444841e-15 -1.5707963267947766539
- joint left_shoulder_pitch: limit lower=-2.1816615649929120835 upper=2.1816615649929120835 effort=10 velocity=6 -> effort=10 velocity=6; origin xyz=0.03086897349438466609 0.079500000000020845659 0.14300000000001039657 rpy=-1.5707963267949047736 -7.2164496600635995543e-15 2.4883110829860584224e-15 -> xyz=0.030868973494384634865 0.079500000000020762392 0.14300000000001031331 rpy=-1.5707963267949047736 1.5866937393608840934e-15 1.2760953914789753679e-15
- joint left_shoulder_roll: limit lower=-0.087266462599716473902 upper=1.570796326794896558 effort=10 velocity=6 -> effort=10 velocity=6; origin xyz=0.023500000000000003525 0.030000000000000054401 0.034999999999999933942 rpy=-3.1415926535897917837 -1.5707963267948958919 0 -> xyz=0.02350000000000003475 0.029999999999999957256 0.035000000000000100475 rpy=-3.141592653589793116 -1.5707963267948841235 0
- joint right_ankle_pitch: limit lower=-1.570796326794896558 upper=1.570796326794896558 effort=10 velocity=6 -> effort=10 velocity=6; origin xyz=-0.14000000000024515057 -1.5889199678209564581e-14 3.0114799542957371159e-14 rpy=5.0446957243049974607e-16 -6.5007295419637772327e-15 -1.5612511284079219651e-17 -> xyz=-0.14000000000024503954 -1.5279444376403716888e-14 5.0570658771675880416e-14 rpy=-4.4408920984981649157e-16 -2.9422456746621798078e-15 3.0350301903487526264e-14
- joint right_ankle_roll: limit lower=-0.785398163397448279 upper=0.785398163397448279 effort=10 velocity=6 -> effort=10 velocity=6; origin xyz=3.8857805861880478915e-16 0.020099999999999926953 -0.015999999999999691552 rpy=1.570796326794896336 2.4094412794995258621e-15 3.1415926535897926719 -> xyz=-3.3306690738754696213e-16 0.020100000000000037975 -0.016000000000000163397 rpy=1.5707963267948956698 -3.9136528551464144388e-15 3.1415926535897922278
- joint right_elbow: limit lower=-2.7925268031909271649 upper=-0 effort=10 velocity=6 -> effort=10 velocity=6; origin xyz=-0.023500000000009860224 -0.14200000000001986034 -0.0024999999999998911981 rpy=3.141592653589793116 -1.5707963267948954478 0 -> xyz=-0.023500000000010012879 -0.1420000000000199436 -0.0024999999999998703815 rpy=3.141592653589793116 -1.5707963267948956698 0
- joint right_foot_frame: origin xyz=0.05999999999999905409 -0.005500000000000331013 -0.0048299999999974474463 rpy=5.2020940636638788206e-15 -1.570796326794891451 0 -> xyz=0.059999999999999220623 2.9143354396410359186e-16 -0.02032999999999917512 rpy=-3.3006666615197048961e-16 -1.5707963267948956698 0
- joint right_hip_pitch: limit lower=-1.570796326794896558 upper=1.570796326794896558 effort=10 velocity=6 -> effort=10 velocity=6; origin xyz=0.00023594338595557540206 -0.01599999999999995523 -0.020100000000000020628 rpy=1.5707963267949038855 -1.5707963267948861219 0 -> xyz=0.00023594338595563091321 -0.015999999999999979516 -0.020100000000000027567 rpy=1.5707963267948981123 -1.5707963267948947816 0
- joint right_hip_roll: limit lower=-0.52359877559829881566 upper=0.52359877559829881566 effort=10 velocity=6 -> effort=10 velocity=6; origin xyz=4.8572257327350598644e-17 -0.020099054048955403845 -0.06039999999999973862 rpy=1.5707963267949003328 -1.5707963267948901187 0 -> xyz=-2.3592239273284576484e-16 -0.020099054048956514068 -0.060400000000000696188 rpy=1.5707963267948976682 -1.5707963267948952257 0
- joint right_hip_yaw: limit lower=-1.0471975511965976313 upper=1.0471975511965976313 effort=10 velocity=6 -> effort=10 velocity=6; origin xyz=0.0058689734943568345332 -0.046400000000004472389 -0.041099999999999956013 rpy=3.9664277854914981584e-16 -5.2373734976912576551e-15 1.5707963267948397146 -> xyz=0.0058689734943574000531 -0.046400000000004514022 -0.041099999999998734768 rpy=2.1625062851527426286e-14 -1.9816742826592979678e-15 1.5707963267948987784
- joint right_knee: limit lower=-0 upper=3.141592653589793116 effort=10 velocity=6 -> effort=10 velocity=6; origin xyz=-2.9143354396410359186e-16 0.14000000000000067946 -9.5756735873919751612e-16 rpy=-3.9621086151768392032e-15 7.7674449885245198315e-16 -1.5707963267948938935 -> xyz=-1.1449174941446926823e-16 0.14000000000000401013 -2.057382042508493214e-14 rpy=1.2767564783171990634e-15 -1.5808749702337738819e-15 -1.5707963267948610309
- joint right_shoulder_pitch: limit lower=-2.1816615649929120835 upper=2.1816615649929120835 effort=10 velocity=6 -> effort=10 velocity=6; origin xyz=0.03086897349437638105 -0.079500000000014198198 0.14300000000001014677 rpy=1.5707963267948708008 -1.8374191057546290257e-14 3.141592653589783346 -> xyz=0.030868973494376360234 -0.079500000000014142687 0.14300000000001011902 rpy=1.5707963267948708008 -4.8017145815038012485e-15 3.141592653589783346
- joint right_shoulder_roll: limit lower=-1.570796326794896558 upper=0.087266462599716473902 effort=10 velocity=6 -> effort=10 velocity=6; origin xyz=-0.023500000000005155654 -0.029999999999999651945 -0.034999999999995798361 rpy=-8.8817841970007218144e-16 -1.5707963267948961139 0 -> xyz=-0.023500000000005162593 -0.029999999999999721334 -0.034999999999995812239 rpy=-3.6082248300526689938e-16 -1.5707963267948750197 0
- joint trunk_frame: origin xyz=0.0058680275433158485265 -3.9238251073735071353e-15 -0.10150000000000060363 rpy=5.5093833584565697626e-15 4.4079575231487197359e-25 -5.958092587816837932e-14 -> xyz=0.0058680275433185069903 -3.8373166558143998956e-15 -0.10150000000000038158 rpy=2.6042242647039365222e-15 -1.132015398992152165e-28 -6.5838035962736754478e-15
